File: receiver/Reciever_Electrical/Reciever_Electrical.kicad_sch (KiCad schematic)
At the start: 0 parts

Commit message: Updated wiring Schematic for Reciever. Added test python scripts.
Parts:
- added D1: POWER (RED), symbol Device:LED
- added D2: GPS LOCK (GREEN), symbol Device:LED
- added D3: RF (BLUE), symbol Device:LED
- added D4: ACTIVITY (YELLOW), symbol Device:LED
- added J1: Raspberry_Pi_5, symbol Connector:Raspberry_Pi_4
- added R1, R2, R3, R4: 220, symbol Device:R_Small_US
Connections:
- new net: D4.1 (K), R4.2
- new net: D4.2 (A), J1.15 (GPIO22/SDIO_CLK)
- new net: D2.1 (K), R2.2
- new net: D1.1 (K), R1.2
- new net: D3.1 (K), R3.2
- new net: D3.2 (A), J1.13 (GPIO27/SDIO_DAT3)
- new net: D2.2 (A), J1.11 (GPIO17/SPI1_~{CE1})
- new net: J1.1 (3V3), J1.17 (3V3)
- new net +5V: D1.2 (A), J1.2 (5V), J1.4 (5V)
- new net GND: J1.14 (GND), J1.20 (GND), J1.25 (GND), J1.30 (GND), J1.34 (GND), J1.39 (GND), J1.6 (GND), J1.9 (GND), R1.1, R2.1, R3.1, R4.1
- new net SCL: J1.5 (SCL_I2C1/GPIO03)
- new net SDA: J1.3 (SDA_I2C1/GPIO02)
- no-connect marks 0 -> 1
Other:
- note added: "NOTE: USB Connections used for: Touchreen Input Controls Touchscreen Power HDMI used for Touchscreen Display."
